File: wallswitch_schematic_alpha/wallswitch_schematic_alpha.sch (KiCad schematic (older format))
At the start: 9 parts

Commit message: schematic - added components
Parts:
- added C? (x2): CP1_Small, symbol Device:CP1_Small
- added C?: C_Small, symbol Device:C_Small
- added F?: Fuse, symbol Device:Fuse
- added R? (x2): R, symbol Device:R
- added RV?: Varistor, symbol Device:Varistor
Connections:
- net labels added: +3V3, +5V, AC_LINE, AC_NEUTRAL, AC_OUT_NC, AC_OUT_NO, GND, RELAY_CTRL
- wire segments 0 -> 45
Other:
- moved on the sheet: J?, K?, PS?, U?

Commit message: added peripheral circuit (50%)
Parts:
- removed C? (x2): CP1_Small, symbol Device:CP1_Small
- removed Q?: 2N7000, Package_TO_SOT_THT:TO-92_Inline, symbol Transistor_FET:2N7000
- added C?: TBD, symbol Device:C_Small
- added C? (x3): 10u, symbol Device:C_Small
- added C? (x2): 0.1u, symbol Device:C_Small
- added C? (x2): 33n, symbol Device:C_Small
- added J?: BOOT, symbol Connector_Generic:Conn_01x02
- added Q? (x2): 2N7002, Package_TO_SOT_SMD:SOT-23, symbol Transistor_FET:2N7002
- added R? (x4): TBD, symbol Device:R
- added R? (x5): 470k 1%, symbol Device:R
- added R?: 1k 1%, symbol Device:R
- added R?: 0, symbol Device:R
- added R? (x2): 15k, symbol Device:R
- added R? (x3): 10k, symbol Device:R
- C?: value C_Small -> 0.1u
Connections:
- net labels added: AC_LINE_IN, AC_LINE_IN_M, GPIO12, GPIO4, GPIO5, RXD, SENSOR_VN, SENSOR_VP, TXD
- wire segments 45 -> 150
Other:
- moved on the sheet: C?, D?, F?, IC?, J?, K?, PS?, R?, RV?, U?

Commit message: updated peripheral circuits
Parts:
- removed J?: BOOT, symbol Connector_Generic:Conn_01x02
- added C?: 10u, symbol Device:C_Small
- added C?: 0.1u, symbol Device:C_Small
- added C? (x2): 1n, symbol Device:C_Small
- added D?: BAT54C, Package_TO_SOT_SMD:SOT-23, symbol Diode:BAT54C
- added D?: LED_3V3, symbol Device:LED_ALT
- added D?: LED_5V, symbol Device:LED_ALT
- added D?: LED_RELAY, symbol Device:LED_ALT
- added J?: Conn_01x06, symbol Connector_Generic:Conn_01x06
- added Q?: BC817DPN, SOT95P275X110-6N, symbol SamacSys_Parts:BC817DPN
- added R?: 10k, symbol Device:R
- added R? (x4): 1k, symbol Device:R
- added R? (x2): 12k, symbol Device:R
- added R? (x2): 470R, symbol Device:R
- added SW?: SW_BOOT, symbol Switch:SW_Push
- added SW?: SW_RESET, symbol Switch:SW_Push
- C?: value TBD -> 1n
- F?: value Fuse -> Fuse 200mA
- R?: value R -> 10k
- R?: value R -> 1k
- R?: value TBD -> 12k
- R? (x2): value TBD -> 1k
- R?: value TBD -> 1m
- RV?: value Varistor -> Varistor 270V
Connections:
- net labels added: 5V_DBG, 5V_TAP, DTR, EN, IO0, IO12, IO13, IO14, IO15, IO16, IO17, IO18, IO19, IO2, IO21, IO22, IO23, IO25, IO26, IO27, IO32, IO33, IO34, IO35, IO4, IO5, RTS, RX, SCK_CLK, SCS_CMD, SDI_SD1, SDO_SD0, SHD_SD2, SWP_SD3, TX
- net labels removed: GPIO12, GPIO4, GPIO5, RELAY_CTRL
- wire segments 150 -> 225
Other:
- note added: "Auto program\nDTR RTS->EN IO0\n 1 1 1 1\n 0 0 1 1\n 1 0 0 1\n 0 1 1 0"
- note added: "Boot Mode Btn"
- note added: "Logic Level\n5V → 3V"
- note added: "RESET Btn"
- note added: "To add:\n1. Capacitive Touch / Manual Switch\n2. Footprint for discrete components"
- moved on the sheet: C?, D?, F?, IC?, J?, K?, PS?, Q?, R?, RV?, U?

Commit message: added components
Parts:
- gave numbers to parts that had none: 60
Other:
- note added: "Auto program:\nDTR RTS | EN IO0\n1 1 1 1\n0 0 1 1\n1 0 0 1\n0 1 1 0"
- note removed: "Auto program\nDTR RTS->EN IO0\n 1 1 1 1\n 0 0 1 1\n 1 0 0 1\n 0 1 1 0"

Commit message: modification of some components to use new XLAB footprint
Parts:
- removed IC1: HLW8012, SOIC127P600X170-8N, symbol SamacSys_Parts:HLW8012
- removed K1: SANYOU_SRD_Form_C, Relay_THT:Relay_SPDT_SANYOU_SRD_Series_Form_C, symbol Relay:SANYOU_SRD_Form_C
- removed PS1: HLK-PM01, Converter_ACDC:Converter_ACDC_HiLink_HLK-PMxx, symbol Converter_ACDC:HLK-PM01
- removed Q1: BC817DPN, SOT95P275X110-6N, symbol SamacSys_Parts:BC817DPN
- added IC1: HLW8012, SOIC127P600X170-8N, symbol XLAB_IC:HLW8012
- added K1: SANYOU_SRD_Form_C, XLAB_Block:Relay_SPDT_SANYOU_SRD_Series_Form_C, symbol XLAB_Block:SANYOU_SRD_Form_C
- added PS1: HLK-PM01, XLAB_Block:Converter_ACDC_HiLink_HLK-PMxx, symbol XLAB_Block:HLK-PM01
- added Q1: BC817DPN, SOT95P275X110-6N, symbol XLAB_IC:BC817DPN
Connections:
- net +5V: now also IC1.1 (VDD), K1.5
- net 5V_TAP: now also PS1.4 (+Vout)
- net AC_LINE_IN_M: now also K1.1
- net AC_NEUTRAL: now also PS1.2 (AC/N)
- net AC_OUT_NC: now also K1.3
- net AC_OUT_NO: now also K1.4
- net DTR: now also Q1.1
- net EN: now also Q1.3
- net GND: now also IC1.5 (GND)
- net IO0: now also Q1.6
- net RTS: now also Q1.4
- net at D4.1 (K), D5.2 (A), Q2.3 (D): now also K1.2
- net at F1.1, RV1.1: now also PS1.1 (AC/L)
- net at C3.2: now also PS1.3 (-Vout)
- net at C9.2, R17.1: now also IC1.2 (V1P)
- net at C10.2, R18.1: now also IC1.3 (V1N)
- net at C11.1, R15.1, R20.2: now also IC1.4 (V2P)
- net at R22.1: now also IC1.6 (CF)
- net at R21.1: now also IC1.7 (CF1)
- net at Q3.3 (D), R24.1: now also IC1.8 (SEL)
- net at R1.1: now also Q1.5
- net at R2.1: now also Q1.2
Changed lines of the file:
@@
 $EndDescr
-$Comp
-L Converter_ACDC:HLK-PM01 PS1
-U 1 1 5EC92670
-P 2800 1100
-F 0 "PS1" H 2800 1425 50  0000 C CNN
-F 1 "HLK-PM01" H 2800 1334 50  0000 C CNN
-F 2 "Converter_ACDC:Converter_ACDC_HiLink_HLK-PMxx" H 2800 800 50  0001 C CNN
-F 3 "http://www.hlktech.net/product_detail.php?ProId=54" H 3200 750 50  0001 C CNN
-	1    2800 1100
-	1    0    0    -1
-$EndComp
 $Comp
 L RF_Module:ESP32-WROOM-32D U2
@@
 F 3 "https://www.espressif.com/sites/default/files/documentation/esp32-wroom-32d_esp32-wroom-32u_datasheet_en.pdf" H 4750 6100 50  0001 C CNN
 	1    5050 6050
-	1    0    0    -1
-$EndComp
-$Comp
-L Relay:SANYOU_SRD_Form_C K1
-U 1 1 5EC90E60
-P 8100 1350
-F 0 "K1" H 8530 1396 50  0000 L CNN
-F 1 "SANYOU_SRD_Form_C" H 8530 1305 50  0000 L CNN
-F 2 "Relay_THT:Relay_SPDT_SANYOU_SRD_Series_Form_C" H 8550 1300 50  0001 L CNN
-F 3 "http://www.sanyourelay.ca/public/products/pdf/SRD.pdf" H 8100 1350 50  0001 C CNN
-	1    8100 1350
 	1    0    0    -1
 $EndComp
@@
 	1    7300 1350
 	0    1    1    0
-$EndComp
-$Comp
-L SamacSys_Parts:HLW8012 IC1
-U 1 1 5ECA7EDE
-P 8350 4600
-F 0 "IC1" H 8850 4865 50  0000 C CNN
-F 1 "HLW8012" H 8850 4774 50  0000 C CNN
-F 2 "SOIC127P600X170-8N" H 9200 4700 50  0001 L CNN
-F 3 "https://www.datasheet4u.com/datasheet-parts/HLW8012-datasheet.php?id=1157559" H 9200 4600 50  0001 L CNN
-F 4 "single phase energy monitor chip" H 9200 4500 50  0001 L CNN "Description"
-F 5 "1.7" H 9200 4400 50  0001 L CNN "Height"
-F 6 "Hilwi" H 9200 4300 50  0001 L CNN "Manufacturer_Name"
-F 7 "HLW8012" H 9200 4200 50  0001 L CNN "Manufacturer_Part_Number"
-F 8 "" H 9200 4100 50  0001 L CNN "Mouser Part Number"
-F 9 "" H 9200 4000 50  0001 L CNN "Mouser Price/Stock"
-F 10 "" H 9200 3900 50  0001 L CNN "RS Part Number"
-F 11 "" H 9200 3800 50  0001 L CNN "RS Price/Stock"
-	1    8350 4600
-	1    0    0    -1
 $EndComp
 Wire Wire Line
@@
 Wire Wire Line
 	1450 6800 1450 6600
-$Comp
-L SamacSys_Parts:BC817DPN Q1
-U 1 1 5F268BD8
-P 1800 6600
-F 0 "Q1" H 1772 6304 50  0000 R CNN
-F 1 "BC817DPN" H 1772 6395 50  0000 R CNN
-F 2 "SOT95P275X110-6N" H 2600 6550 50  0001 L CNN
-F 3 "https://assets.nexperia.com/documents/data-sheet/BC817DPN.pdf" H 2600 6450 50  0001 L CNN
-F 4 "Nexperia BC817DPN Dual NPN+PNP Transistor, 500 mA, 45 V, 6-Pin SOT-457" H 2600 6350 50  0001 L CNN "Description"
-F 5 "1.1" H 2600 6250 50  0001 L CNN "Height"
-F 6 "Nexperia" H 2600 6150 50  0001 L CNN "Manufacturer_Name"
-F 7 "BC817DPN" H 2600 6050 50  0001 L CNN "Manufacturer_Part_Number"
-F 8 "BC817DPN" H 2600 5950 50  0001 L CNN "Arrow Part Number"
-F 9 "" H 2600 5850 50  0001 L CNN "Arrow Price/Stock"
-F 10 "N/A" H 2600 5750 50  0001 L CNN "Mouser Part Number"
-F 11 "https://www.mouser.com/Search/Refine.aspx?Keyword=N%2FA" H 2600 5650 50  0001 L CNN "Mouser Price/Stock"
-	1    1800 6600
-	-1   0    0    1
-$EndComp
 Text Label 700  6800 0    50   ~ 0
 RTS
@@
 Text Notes 650  2450 0    100  ~ 0
 To add:\n1. Capacitive Touch / Manual Switch\n2. Footprint for discrete components
+$Comp
+L XLAB_IC:HLW8012 IC1
+U 1 1 5EFEE691
+P 8350 4600
+F 0 "IC1" H 8850 4865 50  0000 C CNN
+F 1 "HLW8012" H 8850 4774 50  0000 C CNN
+F 2 "SOIC127P600X170-8N" H 9200 4700 50  0001 L CNN
+F 3 "https://www.datasheet4u.com/datasheet-parts/HLW8012-datasheet.php?id=1157559" H 9200 4600 50  0001 L CNN
+F 4 "single phase energy monitor chip" H 9200 4500 50  0001 L CNN "Description"
+F 5 "1.7" H 9200 4400 50  0001 L CNN "Height"
+F 6 "Hilwi" H 9200 4300 50  0001 L CNN "Manufacturer_Name"
+F 7 "HLW8012" H 9200 4200 50  0001 L CNN "Manufacturer_Part_Number"
+	1    8350 4600
+	1    0    0    -1
+$EndComp
+$Comp
+L XLAB_IC:BC817DPN Q1
+U 1 1 5EFF0E81
+P 1100 6100
+F 0 "Q1" H 1828 5896 50  0000 L CNN
+F 1 "BC817DPN" H 1828 5805 50  0000 L CNN
+F 2 "SOT95P275X110-6N" H 1900 6050 50  0001 L CNN
+F 3 "https://assets.nexperia.com/documents/data-sheet/BC817DPN.pdf" H 1900 5950 50  0001 L CNN
+F 4 "Nexperia BC817DPN Dual NPN+PNP Transistor, 500 mA, 45 V, 6-Pin SOT-457" H 1900 5850 50  0001 L CNN "Description"
+F 5 "1.1" H 1900 5750 50  0001 L CNN "Height"
+F 6 "Nexperia" H 1900 5650 50  0001 L CNN "Manufacturer_Name"
+F 7 "BC817DPN" H 1900 5550 50  0001 L CNN "Manufacturer_Part_Number"
+F 8 "BC817DPN" H 1900 5450 50  0001 L CNN "Arrow Part Number"
+F 9 "N/A" H 1900 5250 50  0001 L CNN "Mouser Part Number"
+F 10 "https://www.mouser.com/Search/Refine.aspx?Keyword=N%2FA" H 1900 5150 50  0001 L CNN "Mouser Price/Stock"
+	1    1100 6100
+	1    0    0    -1
+$EndComp
+$Comp
+L XLAB_Block:HLK-PM01 PS1
+U 1 1 5F019A58
+P 2800 1100
+F 0 "PS1" H 2800 1425 50  0000 C CNN
+F 1 "HLK-PM01" H 2800 1334 50  0000 C CNN
+F 2 "XLAB_Block:Converter_ACDC_HiLink_HLK-PMxx" H 2800 800 50  0001 C CNN
+F 3 "http://www.hlktech.net/product_detail.php?ProId=54" H 3200 750 50  0001 C CNN
+	1    2800 1100
+	1    0    0    -1
+$EndComp
+$Comp
+L XLAB_Block:SANYOU_SRD_Form_C K1
+U 1 1 5F0765D9
+P 8100 1350
+F 0 "K1" H 8530 1396 50  0000 L CNN
+F 1 "SANYOU_SRD_Form_C" H 8530 1305 50  0000 L CNN
+F 2 "XLAB_Block:Relay_SPDT_SANYOU_SRD_Series_Form_C" H 8550 1300 50  0001 L CNN
+F 3 "http://www.sanyourelay.ca/public/products/pdf/SRD.pdf" H 8100 1350 50  0001 C CNN
+	1    8100 1350
+	1    0    0    -1
+$EndComp
 $EndSCHEMATC

Commit message: 1. Attached appropriate footprint to connectors 2. TODO: Capacitors and varistor
Parts:
- removed D5: 1N4148, Diode_THT:D_DO-35_SOD27_P7.62mm_Horizontal, symbol Diode:1N4148
- removed R1, R2, R7: 12k, symbol Device:R
- removed R10, R21, R22, R24, R26: 10k, symbol Device:R
- removed R12, R13, R14, R15, R16: 470k 1%, symbol Device:R
- removed R17, R18, R27, R3, R4, R8, R9: 1k, symbol Device:R
- removed R19: 0, symbol Device:R
- removed R20: 1k 1%, symbol Device:R
- removed R23, R25: 15k, symbol Device:R
- removed R5, R6: 470R, symbol Device:R
- added D5: 1N4148W, Diode_SMD:D_SOD-123, symbol Diode:1N4148W
- added R1, R2, R7: R_12k_±5%_1608m, R_0603_1608Metric, symbol XLAB_Resistor:R_12k_±5%_1608m
- added R10, R21, R22, R24, R26: R_10k_±5%_1608m, R_0603_1608Metric, symbol XLAB_Resistor:R_10k_±5%_1608m
- added R12, R13, R14, R15, R16: R_470k_±1%_1608m, R_0603_1608Metric, symbol XLAB_Resistor:R_470k_±1%_1608m
- added R17, R18, R27, R3, R4, R8, R9: R_1k_±5%_1608m, R_0603_1608Metric, symbol XLAB_Resistor:R_1k_±5%_1608m
- added R19: R_0_―_1608m, R_0603_1608Metric, symbol XLAB_Resistor:R_0_―_1608m
- added R20: R_1.00k_±1%_1608m, R_0603_1608Metric, symbol XLAB_Resistor:R_1.00k_±1%_1608m
- added R23, R25: R_15k_±5%_1608m, R_0603_1608Metric, symbol XLAB_Resistor:R_15k_±5%_1608m
- added R5, R6: R_470_±5%_1608m, R_0603_1608Metric, symbol XLAB_Resistor:R_470_±5%_1608m
- D1, D2, D4: footprint (none) -> LED_SMD:LED_0603_1608Metric
- J1: footprint (none) -> Connector_PinHeader_2.54mm:PinHeader_1x06_P2.54mm_Vertical
- J2: footprint (none) -> TerminalBlock:TerminalBlock_bornier-2_P5.08mm
- J3: footprint (none) -> TerminalBlock:TerminalBlock_bornier-3_P5.08mm
- SW1, SW2: footprint (none) -> Button_Switch_SMD:SW_SPST_CK_RS282G05A3
Connections:
- net RX is gone; now on net RXD: J1.3 (Pin_3)
- net TX is gone; now on net TXD: J1.2 (Pin_2)
- net +3V3: now also R4.2, R7.1
- net +5V: now also D5.1 (K), R24.1, R3.2, R8.1
- net AC_LINE: now also R18.2
- net AC_LINE_IN_M: now also R17.2, R19.1
- net AC_NEUTRAL: now also R12.1
- net DTR: now also R1.1
- net EN: now also R6.2, R7.2
- net GND: now also R10.2, R19.2, R20.1, R23.2, R25.2, R26.2
- net IO0: now also R5.2
- net IO12: now also R22.1, R23.1
- net IO13: now also R9.2
- net IO4: now also R27.1
- net IO5: now also R21.1, R25.1
- net RTS: now also R2.1
- net at D4.1 (K), K1.2, Q2.3 (D): now also D5.2 (A)
- net at Q2.1 (G): now also R10.1, R9.1
- net at C11.1, IC1.4 (V2P): now also R15.2, R20.2
- net at C9.2, IC1.2 (V1P): now also R17.1
- net at C10.2, IC1.3 (V1N): now also R18.1
- net at IC1.6 (CF): now also R22.2
- net at IC1.7 (CF1): now also R21.2
- net at Q3.1 (G): now also R26.1, R27.2
- net at IC1.8 (SEL), Q3.3 (D): now also R24.2
- net at Q1.2: now also R2.2
- net at Q1.5: now also R1.2
- net at C1.1, SW1.2: now also R5.1
- net at C2.1, SW2.2: now also R6.1
- net at D2.2 (A): now also R4.1
- net at D1.2 (A): now also R3.1
- net at D4.2 (A): now also R8.2
- new net: R12.2, R13.1
- new net: R13.2, R14.2
- new net: R15.1, R16.1
- new net: R14.1, R16.2
Other:
- moved on the sheet: K1

Commit message: progress for layout
Parts:
- added D10, D8: LED_RELAY, LED_SMD:LED_0603_1608Metric, symbol Device:LED_ALT
- added D11, D9: 1N4148W, Diode_SMD:D_SOD-123, symbol Diode:1N4148W
- added D6: LED_USR_1, LED_SMD:LED_0603_1608Metric, symbol Device:LED_ALT
- added D7: LED_USR_2, LED_SMD:LED_0603_1608Metric, symbol Device:LED_ALT
- added H1, H2: MountingHole3.5mm, MountingHole:MountingHole_3.5mm, symbol Mechanical:MountingHole
- added J4: Conn_01x06, Connector_PinHeader_2.54mm:PinHeader_1x06_P2.54mm_Vertical, symbol Connector_Generic:Conn_01x06
- added J5, J6: Screw_Terminal_01x03, TerminalBlock:TerminalBlock_bornier-3_P5.08mm, symbol Connector:Screw_Terminal_01x03
- added K2, K3: SANYOU_SRD_Form_C, XLAB_Block:Relay_SPDT_SANYOU_SRD_Series_Form_C, symbol XLAB_Block:SANYOU_SRD_Form_C
- added Q4, Q5: 2N7002, Package_TO_SOT_SMD:SOT-23, symbol Transistor_FET:2N7002
- added R28, R29: R_470_±5%_1608m, R_0603_1608Metric, symbol XLAB_Resistor:R_470_±5%_1608m
- added R30, R31, R33, R34: R_1k_±5%_1608m, R_0603_1608Metric, symbol XLAB_Resistor:R_1k_±5%_1608m
- added R32, R35: R_10k_±5%_1608m, R_0603_1608Metric, symbol XLAB_Resistor:R_10k_±5%_1608m
- C1, C10, C11, C12, C13, C2, C3, C4, C5, C6, C7, C8, C9: footprint (none) -> Capacitor_SMD:C_0603_1608Metric
- F1: footprint (none) -> Fuse:Fuse_Blade_Mini_directSolder
- R11: footprint (none) -> Resistor_SMD:R_2512_6332Metric_Pad1.52x3.35mm_HandSolder
- RV1: footprint (none) -> Varistor:RV_Disc_D12mm_W3.9mm_P7.5mm
Connections:
- net AC_LINE is gone; now on net AC_LINE_IN: R11.2, R18.2
- net +5V: now also D3.2, K1.2, PS1.4 (+Vout), D11.1 (K), D9.1 (K), K2.2, K3.2, R30.1, R33.1; no longer D3.3, K1.5, U1.3 (VI)
- net AC_LINE_IN: now also J2.1 (Pin_1); no longer J2.2 (Pin_2)
- net AC_NEUTRAL: now also J2.2 (Pin_2), J5.3 (Pin_3), J6.3 (Pin_3); no longer J2.1 (Pin_1)
- net GND: now also C3.2, PS1.3 (-Vout), D6.1 (K), D7.1 (K), J4.6 (Pin_6), Q4.2 (S), Q5.2 (S), R32.2, R35.2
- net at D4.1 (K), D5.2 (A), Q2.3 (D): now also K1.5; no longer K1.2
- net 5V_DBG renamed 5V_EXT
- removed net 5V_TAP: C3.1, D3.2, PS1.4 (+Vout)
- net AC_LINE_IN_M renamed AC_LINE_M
- net AC_LINE_M: now also K2.1, K3.1
- net AC_OUT_NC renamed AC_OUT1_NC
- net AC_OUT1_NC: now also J3.2 (Pin_2); no longer J3.1 (Pin_1)
- net AC_OUT_NO renamed AC_OUT1_NO
- net AC_OUT1_NO: now also J3.1 (Pin_1); no longer J3.2 (Pin_2)
- net EN renamed EN_RESET
- net IO0 renamed BOOT
- net IO12 renamed PMONITOR_CF
- net IO13: no longer names the net of U2.16 (IO13)
- net IO13: no longer R9.2
- net IO14 renamed PMONITOR_CF1
- net PMONITOR_CF1: now also R21.1, R25.1
- net IO15 renamed LED_USR_1
- net LED_USR_1: now also R28.1
- net IO16 renamed REL1_ON
- net REL1_ON: now also R9.2
- net IO17 renamed REL2_ON
- net REL2_ON: now also R31.2
- net IO18: no longer names the net of U2.30 (IO18)
- net IO19: no longer names the net of U2.31 (IO19)
- net IO2 renamed LED_USR_2
- net LED_USR_2: now also R29.1
- net IO21: no longer names the net of U2.33 (IO21)
- net IO22: no longer names the net of U2.36 (IO22)
- net IO23: no longer names the net of U2.37 (IO23)
- net IO25 renamed GPIO25
- net GPIO25: now also J4.1 (Pin_1)
- net IO26: no longer names the net of U2.11 (IO26)
- net IO27 renamed PMONITOR_SEL
- net PMONITOR_SEL: now also R27.1
- net IO32 renamed GPIO32
- net GPIO32: now also J4.3 (Pin_3)
- net IO33 renamed GPIO33
- net GPIO33: now also J4.2 (Pin_2)
- net IO34 renamed GPIO34
- net GPIO34: now also J4.5 (Pin_5)
- net IO35 renamed GPIO35
- net GPIO35: now also J4.4 (Pin_4)
- net IO4: no longer names the net of U2.26 (IO4)
- net IO4: no longer R27.1
- removed net IO5: R21.1, R25.1, U2.29 (IO5)
- net SCK_CLK: no longer names the net of U2.20 (SCK/CLK)
- net SCS_CMD: no longer names the net of U2.19 (SCS/CMD)
- net SDI_SD1: no longer names the net of U2.22 (SDI/SD1)
- net SDO_SD0: no longer names the net of U2.21 (SDO/SD0)
- net SENSOR_VN: no longer names the net of U2.5 (SENSOR_VN)
- net SENSOR_VP: no longer names the net of U2.4 (SENSOR_VP)
- net SHD_SD2: no longer names the net of U2.17 (SHD/SD2)
- net SWP_SD3: no longer names the net of U2.18 (SWP/SD3)
- new net: C3.1, D3.3, U1.3 (VI)
- new net: D6.2 (A), R28.2
- new net: D7.2 (A), R29.2
- new net: D8.1 (K), D9.2 (A), K2.5, Q4.3 (D)
- new net: D8.2 (A), R30.2
- new net: Q4.1 (G), R31.1, R32.1
- new net: D10.1 (K), D11.2 (A), K3.5, Q5.3 (D)
- new net: D10.2 (A), R33.2
- new net: Q5.1 (G), R34.1, R35.1
- new net AC_OUT2_NC: J5.2 (Pin_2), K2.3
- new net AC_OUT2_NO: J5.1 (Pin_1), K2.4
- new net AC_OUT3_NC: J6.2 (Pin_2), K3.3
- new net AC_OUT3_NO: J6.1 (Pin_1), K3.4
- new net REL3_ON: R34.2, U2.29 (IO5)
- no-connect marks 0 -> 14
Other:
- note added: "Auto program:\nDTR RTS | EN BOOT\n1 1 1 1\n0 0 1 1\n1 0 0 1\n0 1 1 0"
- note added: "Logic Level\n5V → 3V3"
- note removed: "Auto program:\nDTR RTS | EN IO0\n1 1 1 1\n0 0 1 1\n1 0 0 1\n0 1 1 0"
- note removed: "Logic Level\n5V → 3V"
- note removed: "To add:\n1. Capacitive Touch / Manual Switch\n2. Footprint for discrete components"
- moved on the sheet: C1, C10, C11, C12, C13, C2, C3, C4, C5, C6, C7, C8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
