File: wallswitch_schematic_alpha/wallswitch_schematic_alpha.sch (KiCad schematic (older format))
At the start: 84 parts, among them IC1 HLW8012, J1 Conn_01x06, J2 Screw_Terminal_01x02, J3 Screw_Terminal_01x03, J4 Conn_01x06, J5 Screw_Terminal_01x03, J6 Screw_Terminal_01x03, K1 SANYOU_SRD_Form_C, K2 SANYOU_SRD_Form_C, K3 SANYOU_SRD_Form_C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

Commit message: modification to generate gerber files
Parts:
- removed H1, H2: MountingHole3.5mm, MountingHole:MountingHole_3.5mm, symbol Mechanical:MountingHole
Changed lines of the file:
@@
 	7500 5250 7400 5250
-$Comp
-L Mechanical:MountingHole H1
-U 1 1 5F9F9252
-P 9250 1900
-F 0 "H1" H 9350 1946 50  0000 L CNN
-F 1 "MountingHole3.5mm" H 9350 1855 50  0000 L CNN
-F 2 "MountingHole:MountingHole_3.5mm" H 9250 1900 50  0001 C CNN
-F 3 "~" H 9250 1900 50  0001 C CNN
-	1    9250 1900
-	1    0    0    -1
-$EndComp
-$Comp
-L Mechanical:MountingHole H2
-U 1 1 5FA0CC98
-P 9250 2150
-F 0 "H2" H 9350 2196 50  0000 L CNN
-F 1 "MountingHole3.5mm" H 9350 2105 50  0000 L CNN
-F 2 "MountingHole:MountingHole_3.5mm" H 9250 2150 50  0001 C CNN
-F 3 "~" H 9250 2150 50  0001 C CNN
-	1    9250 2150
-	1    0    0    -1
-$EndComp
 $Comp
 L power:GND #PWR0129
